Commit message: adding better repo organization

File: ros2/two_finger_gripper/models/two_finger_gripper.urdf (robot description, URDF)
Before this commit: robot two_link_manipulator, 9 links, 8 joints
Links:
- removed link palm
- added link base, mass 0.187618707682634; collision mesh filename=package://two_finger_gripper/meshes/palm.STL; visual mesh filename=package://two_finger_gripper/meshes/palm.STL
- link LL1: mass 0.049843 -> 0.0498429374208328; geometry collision mesh filename=package://two_finger_gripper/meshes/LL1.STL; visual mesh filename=package://two_finger_gripper/meshes/LL1.STL
- link LL2: mass 0.043363 -> 0.0433629505400265; geometry collision mesh filename=package://two_finger_gripper/meshes/LL2.STL; visual mesh filename=package://two_finger_gripper/meshes/LL2.STL
- link LL3: mass 0.042971 -> 0.0429708569563452; geometry collision mesh filename=package://two_finger_gripper/meshes/LL3.STL; visual mesh filename=package://two_finger_gripper/meshes/LL3.STL
- link Left_base: mass 0.0040046 -> 0.00400455448945672; geometry collision mesh filename=package://two_finger_gripper/meshes/Left_base.STL; visual mesh filename=package://two_finger_gripper/meshes/Left_base.STL
- link RL1: mass 0.049843 -> 0.0498429795113518; geometry collision mesh filename=package://two_finger_gripper/meshes/RL1.STL; visual mesh filename=package://two_finger_gripper/meshes/RL1.STL
- link RL2: mass 0.043363 -> 0.0433629505400265; geometry collision mesh filename=package://two_finger_gripper/meshes/RL2.STL; visual mesh filename=package://two_finger_gripper/meshes/RL2.STL
- link RL3: mass 0.042971 -> 0.0429708583079173; geometry collision mesh filename=package://two_finger_gripper/meshes/RL3.STL; visual mesh filename=package://two_finger_gripper/meshes/RL3.STL
- link Right_base: mass 0.0040046 -> 0.00400455448945673; geometry collision mesh filename=package://two_finger_gripper/meshes/Right_base.STL; visual mesh filename=package://two_finger_gripper/meshes/Right_base.STL
Joints:
- joint joint1: origin xyz=0.61073 -1.3084 0.89978 rpy=1.5708 0 -0.77764 -> xyz=-0.057418 -0.016597 -5.4093E-05 rpy=-3.1416 0.0062462 3.1416; parent palm -> base; type revolute -> continuous
- joint joint2: axis 0 0 1 -> -0.0067813 0 0.99998; origin xyz=0 0.01 0 rpy=0 0 -0.66305 -> xyz=0.032238 0.0036282 0 rpy=3.1416 -0.0067813 -2.7416
- joint joint3: axis 0 0 1 -> 0 0 0; origin xyz=-0.07 0 0 rpy=0 0 0.95183 -> xyz=-0.048792 0.026641 -0.00033088 rpy=-0.0026405 -0.0062461 0.39996; type revolute -> fixed
- joint joint4: origin xyz=0.06 0 0 rpy=0 0 0.91379 -> xyz=0.008449 0.052466 0 rpy=0 0 0
- joint joint5: origin xyz=0.73083 -1.3084 0.89978 rpy=1.5708 0 2.9852 -> xyz=0.0626776436313551 -0.016597406252991 -5.40925989244405E-05 rpy=3.14159265358979 0.0120396735067157 -3.14159265358979; parent palm -> base; type revolute -> continuous
- joint joint6: origin xyz=0 0.01 0 rpy=0 0 1.9755 -> xyz=-0.0299298995045382 0.00814390023253674 0 rpy=3.14159265358979 0 -3.14159265358979
- joint joint7: origin xyz=0.07 0 0 rpy=0 0 -0.77973 -> xyz=0.0253746560766339 0.0477960461466609 0 rpy=0 0 0
- joint joint8: origin xyz=0.06 0 0 rpy=0 0 0.78605 -> xyz=-0.011920133812663 0.0535426961300677 0 rpy=0 0 0

Commit message: URDF fixed

File: ros2/two_finger_gripper/models/two_finger_gripper.urdf (robot description, URDF)
Before this commit: robot two_finger_gripper, 9 links, 8 joints
Links:
- removed link LL1
- removed link LL2
- removed link LL3
- removed link Left_base
- removed link RL1
- removed link RL2
- removed link RL3
- removed link Right_base
- removed link base
- added link L1, mass 0.0498429374208329; collision mesh filename=package://two_finger_gripper/meshes/L1.STL; visual mesh filename=package://two_finger_gripper/meshes/L1.STL
- added link L2, mass 0.0433629505400265; collision mesh filename=package://two_finger_gripper/meshes/L2.STL; visual mesh filename=package://two_finger_gripper/meshes/L2.STL
- added link L3, mass 0.0429708569563452; collision mesh filename=package://two_finger_gripper/meshes/L3.STL; visual mesh filename=package://two_finger_gripper/meshes/L3.STL
- added link R1, mass 0.0498429795113518; collision mesh filename=package://two_finger_gripper/meshes/R1.STL; visual mesh filename=package://two_finger_gripper/meshes/R1.STL
- added link R2, mass 0.0433629505400265; collision mesh filename=package://two_finger_gripper/meshes/R2.STL; visual mesh filename=package://two_finger_gripper/meshes/R2.STL
- added link R3, mass 0.0429708583079173; collision mesh filename=package://two_finger_gripper/meshes/R3.STL; visual mesh filename=package://two_finger_gripper/meshes/R3.STL
- added link base_link, mass 0.187618707682634; collision mesh filename=package://two_finger_gripper/meshes/base_link.STL; visual mesh filename=package://two_finger_gripper/meshes/base_link.STL
- added link left_side, mass 0.00400455448945672; collision mesh filename=package://two_finger_gripper/meshes/left_side.STL; visual mesh filename=package://two_finger_gripper/meshes/left_side.STL
- added link right_side, mass 0.00400455448945673; collision mesh filename=package://two_finger_gripper/meshes/right_side.STL; visual mesh filename=package://two_finger_gripper/meshes/right_side.STL
Joints:
- removed joint joint1
- removed joint joint2
- removed joint joint3
- removed joint joint4
- removed joint joint5
- removed joint joint6
- removed joint joint7
- removed joint joint8
- added joint L1_joint: type revolute, parent left_side, child L1, origin xyz=0 0 0.009 rpy=0 0 0, axis 1 0 0, limit lower=-0.5235 upper=1.57 effort=10.0 velocity=4.0
- added joint L2_joint: type revolute, parent L1, child L2, origin xyz=0 0 0.07 rpy=0 0 0, axis 1 0 0, limit lower=-2 upper=1.57 effort=10.0 velocity=4.0
- added joint L3_joint: type revolute, parent L2, child L3, origin xyz=0 0 0.06 rpy=0 0 0, axis 1 0 0, limit lower=-1.57 upper=0.5235 effort=10.0 velocity=4.0
- added joint R1_joint: type revolute, parent right_side, child R1, origin xyz=0 0.0 0.009 rpy=0 0 0, axis 1 0 0, limit lower=-1.57 upper=0.5235 effort=10.0 velocity=4.0
- added joint R2_joint: type revolute, parent R1, child R2, origin xyz=0 0.0 0.07 rpy=0 0 0, axis 1 0 0, limit lower=-0.5235 upper=2 effort=10.0 velocity=4.0
- added joint R3_joint: type revolute, parent R2, child R3, origin xyz=0 0 0.06 rpy=0 0 0, axis 1 0 0, limit lower=-0.5235 upper=1.57 effort=10.0 velocity=4.0
- added joint left_base_joint: type revolute, parent base_link, child left_side, origin xyz=0 -0.060046 0.015 rpy=0 0 0, axis 0 0 1, limit lower=-0.5235 upper=0.5235 effort=10.0 velocity=4.0
- added joint right_base_joint: type revolute, parent base_link, child right_side, origin xyz=0 0.06005 0.015 rpy=0 0 0, axis 0 0 1, limit lower=-0.5235 upper=0.5235 effort=10.0 velocity=4.0

Commit message: final URDF

File: ros2/two_finger_gripper/models/two_finger_gripper.urdf (robot description, URDF)
Before this commit: robot two_finger_gripper, 9 links, 8 joints
Links:
- added link left_side_pitch, mass 0.00400455448945672; collision mesh filename=package://two_finger_gripper/meshes/left_side.STL; visual mesh filename=package://two_finger_gripper/meshes/left_side.STL
- added link right_side_pitch, mass 0.00400455448945672; collision mesh filename=package://two_finger_gripper/meshes/right_side.STL; visual mesh filename=package://two_finger_gripper/meshes/right_side.STL
Joints:
- removed joint left_base_joint
- added joint left_base_pitch_joint: type revolute, parent left_side, child left_side_pitch, origin xyz=0 0 0.025 rpy=0 0 0, axis 0 1 0, limit lower=-0.5235 upper=0.5235 effort=10.0 velocity=4.0
- added joint left_base_yaw_joint: type revolute, parent base_link, child left_side, origin xyz=0 -0.060046 0.015 rpy=0 0 0, axis 0 0 1, limit lower=-0.5235 upper=0.5235 effort=10.0 velocity=4.0
- added joint right_base_pitch_joint: type revolute, parent right_side, child right_side_pitch, origin xyz=0 0 0.025 rpy=0 0 0, axis 0 1 0, limit lower=-0.5235 upper=0.5235 effort=10.0 velocity=4.0
- joint L1_joint: parent left_side -> left_side_pitch
- joint R1_joint: parent right_side -> right_side_pitch
